Commit message: Added solo6 and mjcf files

File: src/robot_properties_solo/resources/xacro/leg.xacro (robot description, xacro)
@@ -48,5 +48,5 @@
             <xacro:unless value="${is_right}">
                 <xacro:if value="${is_front}">
-                    <origin xyz="0.01950 0 0" rpy="0 0 0" />
+                    <origin xyz="0.0 0 0" rpy="0 0 0" />
                     <geometry>
                         <mesh filename="package://robot_properties_solo/resources/meshes/${mesh_ext}/solo12/solo12_hip_fe_fl.${mesh_ext}"/>
@@ -54,5 +54,5 @@
                 </xacro:if>
                 <xacro:unless value="${is_front}">
-                    <origin xyz="-0.01950 0 0" rpy="0 0 0" />
+                    <origin xyz="-0.0 0 0" rpy="0 0 0" />
                     <geometry>
                         <mesh filename="package://robot_properties_solo/resources/meshes/${mesh_ext}/solo12/solo12_hip_fe_hl.${mesh_ext}"/>
@@ -62,5 +62,5 @@
             <xacro:if value="${is_right}">
                 <xacro:if value="${is_front}">
-                    <origin xyz="0.01950 0 0" rpy="0 0 0" />
+                    <origin xyz="0.0 0 0" rpy="0 0 0" />
                     <geometry>
                         <mesh filename="package://robot_properties_solo/resources/meshes/${mesh_ext}/solo12/solo12_hip_fe_fr.${mesh_ext}"/>
@@ -68,5 +68,5 @@
                 </xacro:if>
                 <xacro:unless value="${is_front}">
-                    <origin xyz="-0.01950 0 0" rpy="0 0 0" />
+                    <origin xyz="-0.0 0 0" rpy="0 0 0" />
                     <geometry>
                         <mesh filename="package://robot_properties_solo/resources/meshes/${mesh_ext}/solo12/solo12_hip_fe_hr.${mesh_ext}"/>
@@ -82,5 +82,5 @@
                 <xacro:unless value="${is_right}">
                 <xacro:if value="${is_front}">
-                    <origin xyz="0.01950 0 0" rpy="0 0 0" />
+                    <origin xyz="0.0 0 0" rpy="0 0 0" />
                     <geometry>
                         <mesh filename="package://robot_properties_solo/resources/meshes/${mesh_ext}/solo12/solo12_hip_fe_fl.${mesh_ext}"/>
@@ -88,5 +88,5 @@
                 </xacro:if>
                 <xacro:unless value="${is_front}">
-                    <origin xyz="-0.01950 0 0" rpy="0 0 0" />
+                    <origin xyz="-0.0 0 0" rpy="0 0 0" />
                     <geometry>
                         <mesh filename="package://robot_properties_solo/resources/meshes/${mesh_ext}/solo12/solo12_hip_fe_hl.${mesh_ext}"/>
@@ -96,5 +96,5 @@
             <xacro:if value="${is_right}">
                 <xacro:if value="${is_front}">
-                    <origin xyz="0.01950 0 0" rpy="0 0 0" />
+                    <origin xyz="0.0 0 0" rpy="0 0 0" />
                     <geometry>
                         <mesh filename="package://robot_properties_solo/resources/meshes/${mesh_ext}/solo12/solo12_hip_fe_fr.${mesh_ext}"/>
@@ -102,5 +102,5 @@
                 </xacro:if>
                 <xacro:unless value="${is_front}">
-                    <origin xyz="-0.01950 0 0" rpy="0 0 0" />
+                    <origin xyz="-0.0 0 0" rpy="0 0 0" />
                     <geometry>
                         <mesh filename="package://robot_properties_solo/resources/meshes/${mesh_ext}/solo12/solo12_hip_fe_hr.${mesh_ext}"/>

Commit message: Added solo13  and updated mjcf files

File: src/robot_properties_solo/resources/xacro/leg.xacro (robot description, xacro)
@@ -14,9 +14,9 @@
   <xacro:property name="KFE_2_FOOT_z" value="${160.00 * 0.001}" />
   <!-- Macro defining solo leg. -->
-  <xacro:macro name="leg" params="prefix is_front is_right has_side_motion
+  <xacro:macro name="leg" params="prefix parent:=base_link is_front is_right has_side_motion
                                   mesh_ext color_name color opacity">
     <xacro:if value="${has_side_motion}">
       <joint name="${prefix}_HAA" type="revolute">
-        <parent link="base_link"/>
+        <parent link="${parent}"/>
         <child link="${prefix}_SHOULDER"/>
         <limit effort="1000" lower="-10" upper="10" velocity="1000"/>
