Commit message: Added mjcf xacro to inject environment

File: src/robot_properties_solo/resources/mjcf/solo12.mjcf.xacro (robot description, xacro)
@@ -1,10 +1,18 @@
 <?xml version="1.0"?>
-<mujoco>
+<mujoco xmlns:xacro="http://playerstage.sourceforge.net/gazebo/xmlschema/#interface">
+    <xacro:arg name="environment" default=""/>
+    <xacro:arg name="resources_dir" default= ""/>
     <option cone="elliptic"/>
     <default>
-        <geom solref="0.0125 0.5" solimp= "0.975 0.975 0.001 0.5 2"/>
+        <geom solref="0.002 1" solimp= "0.9 0.985 0.001 0.5 2"/>
     </default>
-    <compiler angle="radian" meshdir="../meshes/stl/solo12/" autolimits="true"/>
+    <compiler angle="radian" meshdir="$(arg resources_dir)/meshes/stl/solo12/" autolimits="true"/>
     <asset>
+        <texture name="grid" type="2d" builtin="checker" rgb1=".1 .2 .3"
+            rgb2=".2 .3 .4" width="300" height="300"/>
+        <material name="grid" texture="grid" texrepeat="8 8" reflectance=".2"/>
+        <texture name="flat" type="2d" builtin="flat"
+            rgb1=".2 .3 .4" width="300" height="300"/>
+        <material name="flat" texture="flat"  reflectance=".2"/>
         <mesh file="solo_12_base.stl"/>
         <mesh file="solo12_hip_fe_fl.stl"/>
@@ -17,4 +25,12 @@
         <mesh file="../without_foot/solo_lower_leg_v2_right_side.stl"/>
     </asset>
+    <xacro:if value="$(eval environment == '')">
+        <worldbody>
+            <geom type="plane" size="4 4 0.1" material="grid"/>
+        </worldbody>
+    </xacro:if>
+    <xacro:unless value="$(eval environment == '')">
+        <include file="$(arg environment)"/>
+    </xacro:unless>
     <worldbody>
         <light diffuse=".5 .5 .5" pos="0 0 3" dir="0 0 -1"/>

Commit message: WIP

File: src/robot_properties_solo/resources/mjcf/solo12.mjcf.xacro (robot description, xacro)
@@ -5,5 +5,5 @@
     <option cone="elliptic"/>
     <default>
-        <geom solref="0.002 1" solimp= "0.9 0.985 0.001 0.5 2"/>
+        <geom solref="0.005 20" solimp= "0.99 0.999 0.002 0.5 2"/>
     </default>
     <compiler angle="radian" meshdir="$(arg resources_dir)/meshes/stl/solo12/" autolimits="true"/>
@@ -44,5 +44,5 @@
                 <inertial mass="0.14196048" pos="-0.09407251 -0.00438935 0.00001384" fullinertia="0.00002802 0.00038264 0.00038050 0.00003687 -0.00000009 0.00000000"/>
                 <body name="FL_UPPER_LEG" pos="-0.0195 0.014 0">
-                    <joint name="FL_HFE" type="hinge" axis="0 1 0" range="-1.45 1.45" damping="0.009" frictionloss="0.005"/>
+                    <joint name="FL_HFE" type="hinge" axis="0 1 0" range="-2.05 2.05" damping="0.009" frictionloss="0.005"/>
                     <geom type="mesh" mesh="solo12_upper_leg_left_side"/>
                     <inertial mass="0.14737324" pos="0.00001530 0.01767640 -0.07838230" fullinertia="0.00041540 0.00041637 0.00002982 0.00000000 -0.00000010 0.00004589"/>
@@ -60,5 +60,5 @@
                 <inertial mass="0.14196048" pos="-0.09407251 0.00438935 -0.00001384" fullinertia="0.00002802 0.00038264 0.00038050 -0.00003687 0.00000009 0.00000000"/>
                 <body name="FR_UPPER_LEG" pos="-0.0195 -0.014 0">
-                    <joint name="FR_HFE" type="hinge" axis="0 1 0" range="-1.45 1.45" damping="0.009" frictionloss="0.005"/>
+                    <joint name="FR_HFE" type="hinge" axis="0 1 0" range="-2.05 2.05" damping="0.009" frictionloss="0.005"/>
                     <geom type="mesh" mesh="solo12_upper_leg_right_side"/>
                     <inertial mass="0.14737324" pos="-0.00001530 -0.01767640 -0.07838230" fullinertia="0.00041540 0.00041637 0.00002982 0.00000000 0.00000010 -0.00004589"/>
@@ -76,5 +76,5 @@
                 <inertial mass="0.14196048" pos="0.09407251 -0.00438935 -0.00001384" fullinertia="0.00002802 0.00038264 0.00038050 -0.00003687 -0.00000009 0.00000000"/>
                 <body name="HL_UPPER_LEG" pos="0.0195 0.014 0">
-                    <joint name="HL_HFE" type="hinge" axis="0 1 0" range="-1.45 1.45" damping="0.009" frictionloss="0.005"/>
+                    <joint name="HL_HFE" type="hinge" axis="0 1 0" range="-2.05 2.05" damping="0.009" frictionloss="0.005"/>
                     <geom type="mesh" mesh="solo12_upper_leg_left_side"/>
                     <inertial mass="0.14737324" pos="0.00001530 0.01767640 -0.07838230" fullinertia="0.00041540 0.00041637 0.00002982 0.00000000 -0.00000010 0.00004589"/>
@@ -92,5 +92,5 @@
                 <inertial mass="0.14196048" pos="0.09407251 0.00438935 0.00001384" fullinertia="0.00002802 0.00038264 0.00038050 0.00003687 0.00000009 0.00000000"/>
                 <body name="HR_UPPER_LEG" pos="0.0195 -0.014 0">
-                    <joint name="HR_HFE" type="hinge" axis="0 1 0" range="-1.45 1.45" damping="0.009" frictionloss="0.005"/>
+                    <joint name="HR_HFE" type="hinge" axis="0 1 0" range="-2.05 2.05" damping="0.009" frictionloss="0.005"/>
                     <geom type="mesh" mesh="solo12_upper_leg_right_side"/>
                     <inertial mass="0.14737324" pos="-0.00001530 -0.01767640 -0.07838230" fullinertia="0.00041540 0.00041637 0.00002982 0.00000000 0.00000010 -0.00004589"/>
